File: KiCad/Klipper Fan Hat.kicad_sch (KiCad schematic)
At the start: 56 parts, among them J1 Vin, J2 Serial, J3 I2C, J4 1 Wire, J5 GPIO5, J6 GPIO6, J7 SPI, J8 GPIO, Q1 IRLML6344, Q2 IRLML6344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

Commit message: update values of pull up resistors
Parts:
- R4, R5, R6: value 3.9k -> 4.7k
Changed lines of the file:
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@@
       (effects (font (size 1.27 1.27)) (justify left))
     )
-    (property "Value" "3.9k" (at 64.9987 135.7693 0)
+    (property "Value" "4.7k" (at 64.9987 135.7693 0)
       (effects (font (size 1.27 1.27)) (justify left))
     )
@@
       (effects (font (size 1.27 1.27)) (justify left))
     )
-    (property "Value" "3.9k" (at 230.0987 140.8493 0)
+    (property "Value" "4.7k" (at 230.0987 140.8493 0)
       (effects (font (size 1.27 1.27)) (justify left))
     )
@@
       (effects (font (size 1.27 1.27)) (justify left))
     )
-    (property "Value" "3.9k" (at 230.0987 111.6393 0)
-      (effects (font (size 1.27 1.27)) (justify left))
-    )
+    (property "Value" "4.7k" (at 230.0987 111.6393 0)
+      (effects (font (size 1.27 1.27)) (justify left))
+    )

Commit message: Update KlippUpdate Klipper Fan Hat to expose more GPIO pins and add an on board DS18B20 Temperature Sensor
Parts:
- removed J5: GPIO5, Connector_JST:JST_XH_B3B-XH-A_1x03_P2.50mm_Vertical, symbol Connector_Generic:Conn_01x03
- removed R5, R6: 4.7k, Resistor_SMD:R_1206_3216Metric, symbol Device:R_Small
- added GPIO20: J7, Connector_PinHeader_2.54mm:PinHeader_1x03_P2.54mm_Vertical, symbol Connector_Generic:Conn_01x03
- added GPIO21: J8, Connector_PinHeader_2.54mm:PinHeader_1x03_P2.54mm_Vertical, symbol Connector_Generic:Conn_01x03
- added GPIO22: J9, Connector_PinHeader_2.54mm:PinHeader_1x03_P2.54mm_Vertical, symbol Connector_Generic:Conn_01x03
- added GPIO24: J11, Connector_PinHeader_2.54mm:PinHeader_1x03_P2.54mm_Vertical, symbol Connector_Generic:Conn_01x03
- added GPIO25: J12, Connector_PinHeader_2.54mm:PinHeader_1x03_P2.54mm_Vertical, symbol Connector_Generic:Conn_01x03
- added U2: DS18B20, Package_TO_SOT_THT:TO-92_Inline, symbol Sensor_Temperature:DS18B20
- GPIO23: renamed from J6; value GPIO6 -> J10; footprint Connector_JST:JST_XH_B3B-XH-A_1x03_P2.50mm_Vertical -> Connector_PinHeader_2.54mm:PinHeader_1x03_P2.54mm_Vertical
- renumbered J7 to J5, J8 to J6
Connections:
- net +3V3: now also GPIO23.2 (Pin_2), GPIO20.2 (Pin_2), GPIO21.2 (Pin_2), GPIO22.2 (Pin_2), GPIO24.2 (Pin_2), GPIO25.2 (Pin_2), U2.3 (V_{DD}); no longer GPIO23.1 (Pin_1)
- net GND: now also GPIO20.3 (Pin_3), GPIO21.3 (Pin_3), GPIO22.3 (Pin_3), GPIO24.3 (Pin_3), GPIO25.3 (Pin_3), U2.1 (GND)
- net GPIO20/PCM.DIN: now also GPIO20.1 (Pin_1)
- net GPIO21/PCM.DOUT: now also GPIO21.1 (Pin_1)
- net GPIO22: now also GPIO22.1 (Pin_1)
- net GPIO23: now also GPIO23.1 (Pin_1)
- net GPIO24: now also GPIO24.1 (Pin_1)
- net GPIO25: now also GPIO25.1 (Pin_1)
- net GPIO4/GPCLK0: now also U2.2 (DQ)
- net GPIO6: no longer GPIO23.2 (Pin_2)
- no-connect marks 12 -> 8
Other:
- moved on the sheet: D6, D7, F1, GPIO23, J1, R1, R22
